File: Kicad/AsicsBoard - 16xBM1368 - 01A/BM1368.kicad_sch (KiCad schematic)
At the start: 23 parts

Commit message: update Hashboard 1368
Parts:
- U4: value ~ -> BM1368
Changed lines of the file:
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@@
 		(on_board yes)
 		(dnp no)
-		(fields_autoplaced yes)
 		(property "Reference" "U4"
 			(at 140.6241 72.39 0)
@@
 			)
 		)
-		(property "Value" "~"
-			(at 141.986 74.93 0)
+		(property "Value" "BM1368"
+			(at 146.05 73.914 0)
 			(effects
 				(font
