File: Kicad/AsicsBoard - 16xBM1368 - 01A/FIXs.kicad_sch (KiCad schematic)
At the start: 40 parts

Commit message: update Hashboard 1368
Parts:
- added C278, C279, C280, C281, C282, C283, C284, C285, C286, C287: 330µF/4V, Capacitor_SMD:C_1210_3225Metric, symbol Device:C_Polarized
Connections:
- net GND: now also C278.2, C279.2, C280.2, C281.2, C282.2, C283.2, C284.2, C285.2, C286.2, C287.2
- net VPWR_ASIC: now also C278.1, C279.1, C280.1, C281.1, C282.1, C283.1, C284.1, C285.1, C286.1, C287.1
Other:
- moved on the sheet: H11, H12, H13, H14, H15, H16, H17, H18, H19, H20, H21, H22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
