File: Kicad/AsicsBoard - 10xBM1370 - 01A/ASICs.kicad_sch (KiCad schematic)
At the start: 13 parts

Commit message: update
Parts:
- R28, R29: P/N MOUSER (none) -> 791-RMC1/16SK103FTH
Changed lines of the file:
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@@
 			)
 		)
-		(property "DK" ""
-			(at 229.87 88.9 0)
-			(effects
-				(font
-					(size 1.27 1.27)
-				)
-				(hide yes)
-			)
-		)
-		(property "PARTNO" ""
+		(property "P/N MOUSER" "791-RMC1/16SK103FTH"
 			(at 229.87 88.9 0)
 			(effects
@@
 			)
 		)
-		(property "DK" ""
+		(property "P/N MOUSER" "791-RMC1/16SK103FTH"
 			(at 71.12 91.44 0)
 			(effects
-				(font
-					(size 1.27 1.27)
-				)
-				(hide yes)
-			)
-		)
-		(property "PARTNO" ""
-			(at 71.12 91.44 0)
-			(effects
