File: Kicad/AsicsBoard - 10xBM1370 - 01A/AsicsBoard - 10xBM1370 - 01A.kicad_pcb (KiCad board)
At the start: 6 copper layers, 139.8 x 65 mm, 319 parts, among them J1 Conn_02x04_Odd_Even, J2 Conn_02x04_Odd_Even, U1 MCP1826S-1202E_DB, U10 BM1370_mode1, U11 BM1370_mode1, U12 BM1370_mode1, U13 BM1370_mode1, U2 MCP1826S-0802E_DB, U3 25MHz, U4 BM1370_mode1, U5 BM1370_mode1, U6 BM1370_mode1, U7 BM1370_mode1, U8 BM1370_mode1, U9 BM1370_mode1

Commit message: update
Parts:
- C1, C2: value 1uF -> 1uF/16V
- C100, C101, C102, C103, C104, C105, C106, C107, C11, C110, C111, C113, C114, C115, C116, C117, C118, C119, C12, C120, C121, C122, C123, C124, C127, C128, C13, C130, C131, C132, C133, C134, C135, C136, C137, C138, C139, C14, C140, C141, C144, C145, C147, C148, C149, C15, C150, C151, C152, C153, C154, C155, C156, C157, C158, C16, C161, C162, C164, C165, C166, C167, C168, C169, C17, C170, C171, C172, C173, C174, C175, C18, C19, C20, C21, C22, C25, C26, C28, C29, C30, C31, C32, C33, C34, C35, C36, C37, C38, C39, C42, C43, C45, C46, C47, C48, C49, C50, C51, C52, C53, C54, C55, C56, C59, C60, C62, C63, C64, C65, C66, C67, C68, C69, C70, C71, C72, C73, C76, C77, C79, C8, C80, C81, C82, C83, C84, C85, C86, C87, C88, C89, C9, C90, C93, C94, C96, C97, C98, C99: value 1uF -> 1uF/6.3V; moved to B.Cu
- C108, C109, C125, C126, C142, C143, C159, C160, C23, C24, C40, C41, C57, C58, C6, C7, C74, C75, C91, C92: moved to B.Cu
- C3, C4: value 1uF -> 100nF; footprint Capacitor_SMD:C_0805_2012Metric_Pad1.18x1.45mm_HandSolder -> Capacitor_SMD:C_0402_1005Metric
- C5: footprint Capacitor_SMD:C_0805_2012Metric_Pad1.18x1.45mm_HandSolder -> Capacitor_SMD:C_0402_1005Metric
- U3: footprint Oscillator:Oscillator_SMD_Abracon_ASE-4Pin_3.2x2.5mm -> EKO_Miner_ASIClib:OSC_SMD_3.2x2.5mm
- moved C104 13.0 mm to (170.5, 107.5)
- moved C107 13.0 mm to (157.5, 107.5)
- moved C155 13.0 mm to (194.5, 107.5)
- moved C158 13.0 mm to (181.5, 107.5)
- moved C19 13.0 mm to (122.5, 107.5)
- moved C22 13.0 mm to (109.5, 107.5)
- moved C36 13.0 mm to (98.5, 107.5)
- moved C39 13.0 mm to (85.5, 107.5)
- moved C70 13.0 mm to (146.5, 107.5)
- moved C73 13.0 mm to (133.5, 107.5)
- moved C121 13.0 mm to (181.5, 67.5)
- moved C124 13.0 mm to (194.5, 67.5)
- moved C138 13.0 mm to (109.5, 67.5)
- moved C141 13.0 mm to (122.5, 67.5)
- moved C172 13.0 mm to (85.5, 67.5)
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Routing:
- net GND: track 206.4 -> 190.3 mm
- net +0.8V: track 383.5 -> 393.9 mm
- net +1.2V: track 385.8 -> 386.3 mm
- net /ASICs/ASICs_BM1370_2/BM1370-4/VDD1_0: track 5.94 -> 6.15 mm, vias 0 -> 1
- net /ASICs/ASICs_BM1370_2/BM1370-3/VDD1_1: track 5.94 -> 6.15 mm, vias 0 -> 1
- net /ASICs/ASICs_BM1370_2/BM1370-3/VDD1_0: track 5.94 -> 6.15 mm, vias 0 -> 1
- net /ASICs/ASICs_BM1370_1/BM1370-0/VDD1_0: track 5.94 -> 6.15 mm, vias 0 -> 1
- net /ASICs/ASICs_BM1370_2/BM1370-4/VDD1_1: track 5.94 -> 6.15 mm, vias 0 -> 1
- net /ASICs/ASICs_BM1370_2/BM1370-2/VDD1_1: track 5.94 -> 6.15 mm, vias 0 -> 1
- net /ASICs/ASICs_BM1370_2/BM1370-2/VDD1_0: track 5.94 -> 6.15 mm, vias 0 -> 1
- net /ASICs/ASICs_BM1370_2/BM1370-1/VDD1_1: track 5.94 -> 6.15 mm, vias 0 -> 1
- net /ASICs/ASICs_BM1370_2/BM1370-1/VDD1_0: track 5.94 -> 6.15 mm, vias 0 -> 1
- net /ASICs/ASICs_BM1370_2/BM1370-0/VDD1_1: track 5.94 -> 6.15 mm, vias 0 -> 1
- net /ASICs/ASICs_BM1370_2/BM1370-0/VDD1_0: track 5.94 -> 6.15 mm, vias 0 -> 1
- net /ASICs/ASICs_BM1370_1/BM1370-4/VDD1_1: track 5.94 -> 6.15 mm, vias 0 -> 1
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Other:
- board text added: "6"
