File: Kicad/AsicsBoard - 10xBM1370 - 01A/AsicsBoard - 10xBM1370 - 01A.kicad_sch (KiCad schematic)
At the start: 16 parts, among them J1 Conn_02x04_Odd_Even, J2 Conn_02x04_Odd_Even, U1 MCP1826S-1202E_DB, U2 MCP1826S-0802E_DB, U3 25MHz

Commit message: update
Parts:
- C1, C2: value 1uF -> 1uF/16V; P/N MOUSER (none) -> 187-CL21B105KOFNFNE
- C3, C4: value 1uF -> 100nF; footprint Capacitor_SMD:C_0805_2012Metric_Pad1.18x1.45mm_HandSolder -> Capacitor_SMD:C_0402_1005Metric; P/N MOUSER (none) -> 791-SH15B104K160CT
- C5: footprint Capacitor_SMD:C_0805_2012Metric_Pad1.18x1.45mm_HandSolder -> Capacitor_SMD:C_0402_1005Metric; P/N MOUSER (none) -> 791-SH15B104K160CT
- J1, J2: P/N MOUSER (none) -> 649-1012938390801ALF
- R1, R2: P/N MOUSER (none) -> 603-RT0805DRE0751RL
- U1, U2: SnapEDA_Link https://www.snapeda.com/parts/MCP1826S-1802E/DB/Microchip/v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 -> (none)
- U3: footprint Oscillator:Oscillator_SMD_Abracon_ASE-4Pin_3.2x2.5mm -> EKO_Miner_ASIClib:OSC_SMD_3.2x2.5mm; P/N MOUSER (none) -> 449-LFSPXO076024CUTT
