File: Kicad/AsicsBoard - 10xBM1370 - 01A/BM1370.kicad_sch (KiCad schematic)
At the start: 23 parts, among them U10 BM1370_mode1

Commit message: update
Parts:
- C108, C109: DK 1292-1639-1-ND -> (none); P/N MOUSER (none) -> 791-SH15B104K160CT; PARTNO 0402X104K100CT -> (none)
- C110, C111, C113, C114, C115, C116, C117, C118, C119, C120, C121, C122, C123, C124: value 1uF -> 1uF/6.3V; DK 587-5514-1-ND -> (none); P/N MOUSER (none) -> 81-GRM155R70J105KA2D; PARTNO EMK105BJ105MV-F -> (none)
- R35, R36, R37, R38: DK 311-33.0LRCT-ND -> (none); P/N MOUSER (none) -> 791-WR04X33R0FTL; PARTNO RC0402FR-0733RL -> (none)
- R39: P/N MOUSER (none) -> 708-RNCP0402FTD1K00
