File: Kicad/PowerBoard TPS53667/EKO_Miner_PowerBoard-53667.kicad_sch (KiCad schematic)
At the start: 17 parts, among them J1 10018784-10210TLF, J2 10018784-10210TLF, J3 Conn_02x04_Odd_Even, J4 Conn_02x04_Odd_Even, J9 Conn_01x03, U2 SN74AXC4T245BQB

Commit message: update
Parts:
- D1: P/N MOUSER (none) -> 859-LTST-C171GKT
- J1, J2: value 10018784-10210TLF -> PCB 10018784-10210TLF; MP 10018784-10210TLF -> (none); now left out of the parts list
- J3, J4: footprint Connector_Wuerth:Wuerth_WR-PHD_610008243021_SMD_2x04_P2.54mm_Vertical -> EKO_Miner_ASIClib:M20_7810445; P/N MOUSER (none) -> 855-M20-7810445
- U2: P/N MOUSER (none) -> 595-SN74AXC4T245BQBR
Changed lines of the file:
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@@
 			)
 		)
-		(property "Footprint" "Connector_Wuerth:Wuerth_WR-PHD_610008243021_SMD_2x04_P2.54mm_Vertical"
+		(property "Footprint" "EKO_Miner_ASIClib:M20_7810445"
 			(at 250.19 58.42 0)
 			(effects
@@
 			)
 		)
+		(property "P/N MOUSER" "855-M20-7810445"
+			(at 250.19 58.42 0)
+			(effects
+				(font
+					(size 1.27 1.27)
+				)
+				(hide yes)
+			)
+		)
 		(pin "1"
 		)
@@
 			)
 		)
-		(property "Footprint" "Connector_Wuerth:Wuerth_WR-PHD_610008243021_SMD_2x04_P2.54mm_Vertical"
+		(property "Footprint" "EKO_Miner_ASIClib:M20_7810445"
 			(at 246.38 142.24 0)
 			(effects
@@
 			)
 		)
+		(property "P/N MOUSER" "855-M20-7810445"
+			(at 246.38 142.24 0)
+			(effects
+				(font
+					(size 1.27 1.27)
+				)
+				(hide yes)
+			)
+		)
 		(pin "1"
 		)
@@
 			)
 		)
+		(property "P/N MOUSER" "859-LTST-C171GKT"
+			(at 87.63 172.72 0)
+			(effects
+				(font
+					(size 1.27 1.27)
+				)
+				(hide yes)
+			)
+		)
 		(pin "2"
 		)
@@
 		(at 49.53 102.87 0)
 		(unit 1)
-		(exclude_from_sim no)
-		(in_bom yes)
+		(exclude_from_sim yes)
+		(in_bom no)
 		(on_board yes)
 		(dnp no)
@@
 			)
 		)
-		(property "Value" "10018784-10210TLF"
+		(property "Value" "PCB 10018784-10210TLF"
 			(at 49.53 74.93 0)
 			(effects
@@
 			)
 		)
-		(property "MP" "10018784-10210TLF"
-			(at 49.53 102.87 0)
-			(effects
-				(font
-					(size 1.27 1.27)
-				)
-				(justify bottom)
-				(hide yes)
-			)
-		)
 		(property "Purchase-URL" "https://www.snapeda.com/api/url_track_click_mouser/?unipart_id=520950&manufacturer=Amphenol ICC&part_name=10018784-10210TLF&search_term=10018784-10210tlf"
 			(at 49.53 102.87 0)
@@
 		(at 49.53 45.72 0)
 		(unit 1)
-		(exclude_from_sim no)
-		(in_bom yes)
+		(exclude_from_sim yes)
+		(in_bom no)
 		(on_board yes)
 		(dnp no)
@@
 			)
 		)
-		(property "Value" "10018784-10210TLF"
+		(property "Value" "PCB 10018784-10210TLF"
 			(at 49.53 17.78 0)
 			(effects
@@
 			)
 		)
-		(property "MP" "10018784-10210TLF"
-			(at 49.53 45.72 0)
-			(effects
-				(font
-					(size 1.27 1.27)
-				)
-				(justify bottom)
-				(hide yes)
-			)
-		)
 		(property "Purchase-URL" "https://www.snapeda.com/api/url_track_click_mouser/?unipart_id=520950&manufacturer=Amphenol ICC&part_name=10018784-10210TLF&search_term=10018784-10210tlf"
 			(at 49.53 45.72 0)
@@
 			(at 142.24 137.16 0)
 			(effects
+				(font
+					(size 1.27 1.27)
+				)
+				(hide yes)
+			)
+		)
+		(property "P/N MOUSER" "595-SN74AXC4T245BQBR"
+			(at 142.24 137.16 0)
+			(effects
