File: Kicad/PowerBoard TPS53667/FAN.kicad_sch (KiCad schematic)
At the start: 16 parts, among them J5 Conn_01x04, J6 Conn_01x04, U3 MAX6615AEE_

Commit message: update
Parts:
- U3: P/N MOUSER (none) -> 700-MAX6615AEE
Changed lines of the file:
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@@
+			)
+		)
+		(property "P/N MOUSER" "700-MAX6615AEE"
+			(at 96.52 99.06 0)
+			(effects
+				(font
+					(size 1.27 1.27)
+				)
+				(hide yes)
 			)
 		)
