File: Kicad/PowerBoard TPS53667/PSU_53667.kicad_sch (KiCad schematic)
At the start: 80 parts, among them J7 Conn_01x01, J8 Conn_01x01, Q1 BSS138, Q2 BSS138, U4 TPS53667RTAR

Commit message: update
Parts:
- C103, C63, C68, C72, C77, C82, C86, C90, C94, C99: value 10uF -> 10uF/25V; P/N MOUSER (none) -> 963-TMK212BBJ106MG-T
- C19, C40: P/N MOUSER (none) -> 603-CC805KRX7R0BB102
- C31: value 4.7µF -> 4.7µF/16V; P/N MOUSER (none) -> 187-CL21A475KOFNNNG
- C32, C33: P/N MOUSER (none) -> 187-CL21B105KAFNNNE
- C36: P/N MOUSER (none) -> 187-CL21B334KBFNNNE
- C38: P/N MOUSER (none) -> 581-KGM15ACG2A120JM
- C41: P/N MOUSER (none) -> 791-0805B222K160CT
- C56, C58, C61, C62, C64, C67, C69, C71, C74, C76: value 100uF/4V -> 100uF/6.3V; P/N MOUSER 963-AMK316ABJ107ML-T -> 187-CL31A107MQHNNWE
- D2: P/N MOUSER (none) -> 859-LTST-C171GKT
- R11, R12: P/N MOUSER (none) -> 603-RT0805DRE0751RL
- R14: P/N MOUSER (none) -> 603-RT0805FRE07121KL
- R19: P/N MOUSER (none) -> 603-RC0805FR-0716K5L
- R20: P/N MOUSER (none) -> 603-RC0805FR-0724K3L
- R22: P/N MOUSER (none) -> 667-ERJ-P06F2551V
- R23, R24: value 2.2R/0.5W -> 2.2R
- R25: P/N MOUSER (none) -> 603-RC0805FR-078K06L
- R26: value 100k -> 100K; P/N MOUSER (none) -> 279-CRG0805F100K
- R27: value 49.9k -> 49.9K; P/N MOUSER (none) -> 652-CR0805FX-4992ELF
- R56, R57: P/N MOUSER (none) -> 71-CRCW08050000Z0ECC
- U4: P/N MOUSER (none) -> 595-TPS53667RTAT
