File: Kicad/PowerBoard TPS53667/PowerStage.kicad_sch (KiCad schematic)
At the start: 25 parts, among them U11 CSD95490Q5MC

Commit message: update
Parts:
- added C37, C47: 100uF/6.3V, Capacitor_SMD:C_1206_3216Metric, symbol Device:C
- C115, C116, C138: value 10uF -> 10uF/25V; P/N MOUSER (none) -> 963-TMK212BBJ106MG-T
- C133: value 3.3nF -> 2.2nF; P/N MOUSER (none) -> 791-0805B222K160CT
- C140, C141, C98: P/N MOUSER (none) -> 603-CC805KRX7R0BB102
- C210: P/N MOUSER (none) -> 187-CL21B105KAFNNNE
- L3: P/N MOUSER (none) -> 504-FP1008R5-R220-R
- R32, R49: P/N MOUSER (none) -> 71-CRCW08050000Z0ECC
- R33: P/N MOUSER (none) -> 791-WR08W1R00FTL
- R44: P/N MOUSER (none) -> 279-CRG0805F100K
- U11: P/N MOUSER (none) -> 595-CSD95490Q5MC
Connections:
- net GND: now also C37.2, C47.2
- net VPWR_ASIC: now also C37.1, C47.1
Other:
- moved on the sheet: C115, C116, C144
